Commit message: Model appears in moveit and rviz, but planning does not work

File: workspace/src/robotarm_description/urdf/robotarm.ros2.control.xacro (robot description, xacro)
@@ -15,11 +15,11 @@
             </xacro:unless>
         </xacro:if>
-        <xacro:unless value="$(arg is_sim)">
+        <!-- xacro:unless value="$(arg is_sim)">
             <hardware>
-                <plugin>robotarm_controller/ArduinobotInterface</plugin>
+                <plugin>robotarm_controller/RobotarmInterface</plugin>
                 <param name="port">/dev/ttyUSB0</param>
             </hardware>
-        </xacro:unless>
-        <!-- joint name="joint_1">
+        </xacro:unless -->
+        <joint name="base">
             <command_interface name="position">
                 <param name="min">-${PI /2}</param>
@@ -28,5 +28,5 @@
             <state_interface name="position"/>
         </joint>
-        <joint name="joint_2">
+        <joint name="base_arm1">
             <command_interface name="position">
                 <param name="min">-${PI /2}</param>
@@ -35,5 +35,5 @@
             <state_interface name="position"/>
         </joint>
-        <joint name="joint_3">
+        <joint name="arm1_arm2">
             <command_interface name="position">
                 <param name="min">-${PI /2}</param>
@@ -41,5 +41,12 @@
             </command_interface>
             <state_interface name="position"/>
-        </joint -->
+        </joint>
+        <joint name="arm2_forks">
+            <command_interface name="position">
+                <param name="min">-${PI /2}</param>
+                <param name="max">$PI / 2}</param>
+            </command_interface>
+            <state_interface name="position"/>
+        </joint>
     </ros2_control>
 </robot>

Commit message: Updated code to run via CNC Shield

File: workspace/src/robotarm_description/urdf/robotarm.ros2.control.xacro (robot description, xacro)
@@ -3,5 +3,5 @@
         <xacro:property name="PI" value="3.14159" />
     <ros2_control type="system" name="RobotSystem">
-        <xacro:if value="$(arg is_sim)">
+        <!-- xacro:if value="$(arg is_sim)">
             <xacro:if value="$(arg is_ignition)">
                 <hardware>
@@ -14,15 +14,15 @@
                 </hardware>
             </xacro:unless>
-        </xacro:if>
-        <!-- xacro:unless value="$(arg is_sim)">
+        </xacro:if -->
+        <!-- xacro:unless value="$(arg is_sim)" -->
             <hardware>
                 <plugin>robotarm_controller/RobotarmInterface</plugin>
                 <param name="port">/dev/ttyUSB0</param>
             </hardware>
-        </xacro:unless -->
+        <!-- /xacro:unless -->
         <joint name="base">
             <command_interface name="position">
-                <param name="min">-${PI /2}</param>
-                <param name="max">$PI / 2}</param>
+                <param name="min">-15</param>
+                <param name="max">15</param>
             </command_interface>
             <state_interface name="position"/>
@@ -30,6 +30,6 @@
         <joint name="base_arm1">
             <command_interface name="position">
-                <param name="min">-${PI /2}</param>
-                <param name="max">$PI / 2}</param>
+                <param name="min">-15</param>
+                <param name="max">15</param>
             </command_interface>
             <state_interface name="position"/>
@@ -37,6 +37,6 @@
         <joint name="arm1_arm2">
             <command_interface name="position">
-                <param name="min">-${PI /2}</param>
-                <param name="max">$PI / 2}</param>
+                <param name="min">-15</param>
+                <param name="max">15</param>
             </command_interface>
             <state_interface name="position"/>
@@ -44,6 +44,6 @@
         <joint name="arm2_forks">
             <command_interface name="position">
-                <param name="min">-${PI /2}</param>
-                <param name="max">$PI / 2}</param>
+                <param name="min">-15</param>
+                <param name="max">15</param>
             </command_interface>
             <state_interface name="position"/>

File: workspace/src/robotarm_description/urdf/robotarm.urdf.xacro (robot description, xacro)
@@ -35,5 +35,5 @@
         <parent link="world" />
         <child link="platform_link" />
-        <origin ryp="0 0 0" xyz="${PI/2} 0 0"/>
+        <origin ryp="0 0 0" xyz="15 0 0"/>
     </joint>
     <link name="platform_to_base">
@@ -57,5 +57,5 @@
         <axis xyz="0 0 1" />
         <origin ryp="0 0 0" xyz="0 0 0.307"/>
-        <limit lower="-${PI/2}" upper="${PI/2}" effort="${effort}" velocity="${velocity}"/> <!-- Radians = pi/2 -->
+        <limit lower="-15" upper="15" effort="${effort}" velocity="${velocity}"/> <!-- Radians = pi/2 -->
     </joint>
     <!-- ARM 1 -->
@@ -80,5 +80,5 @@
         <axis xyz="1 0 0" />
         <origin ryp="0 0 0" xyz="0 0 0.95"/>
-        <limit lower="-0.331" upper="${PI/2}" effort="${effort}" velocity="${velocity}"/> <!-- Radians = pi/2 -->
+        <limit lower="-5" upper="5" effort="${effort}" velocity="${velocity}"/> <!-- Radians = pi/2 -->
     </joint>
     <!-- ARM 2 -->
@@ -103,5 +103,5 @@
         <axis xyz="1 0 0" />
         <origin ryp="0 0 0" xyz="0 -0.0125 0.99"/>
-        <limit lower="-${PI/2}" upper="1.149" effort="${effort}" velocity="${velocity}"/> <!-- Radians = pi/2 -->
+        <limit lower="-5" upper="5" effort="${effort}" velocity="${velocity}"/> <!-- Radians = pi/2 -->
     </joint>
     <!-- PALLET FORKS -->
@@ -126,5 +126,5 @@
         <axis xyz="1 0 0" />
         <origin ryp="0 0 0" xyz="0 -1.0 0.0"/>
-        <limit lower="-${PI/2}" upper="0.576" effort="${effort}" velocity="${velocity}"/> <!-- Radians = pi/2 -->
+        <limit lower="-5" upper="5" effort="${effort}" velocity="${velocity}"/> <!-- Radians = pi/2 -->
     </joint>
 </robot>
